File: hardware/eagle/sensor_module.brd (EAGLE design)
At the start: 63.5 x 31.8 mm, 29 parts, among them J1 AVR_SPI_PRG_6PTH, Q1 16MHz, U1 ATMEGA328P, U2 MCP73831

Commit message: Update schematic to latest values and include PDF
Parts:
- C1: value (none) -> 47uF
- C5, C8: value 4.7u -> 4.7uF
- C6, C7: value 22pF -> 18pF
Changed lines of the file:
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@@
 <attribute name="NAME" x="36.957" y="55.245" size="0.6096" layer="25" font="vector" rot="R180"/>
 </element>
-<element name="C1" library="SparkFun-Capacitors" package="EIA3216" value="" x="35.56" y="50.8" smashed="yes" rot="R90">
+<element name="C1" library="SparkFun-Capacitors" package="EIA3216" value="47uF" x="35.56" y="50.8" smashed="yes" rot="R90">
 <attribute name="NAME" x="37.7858" y="48.8188" size="0.6096" layer="25" font="vector" rot="R90"/>
 <attribute name="VALUE" x="34.228" y="51.208" size="0.4064" layer="27" rot="R90"/>
@@
 <attribute name="NAME" x="26.543" y="47.244" size="0.6096" layer="25" font="vector" ratio="10"/>
 </element>
-<element name="C6" library="SparkFun-Capacitors" package="0603-CAP" value="22pF" x="22.86" y="48.514" smashed="yes" rot="R180">
+<element name="C6" library="SparkFun-Capacitors" package="0603-CAP" value="18pF" x="22.86" y="48.514" smashed="yes" rot="R180">
 <attribute name="PROD_ID" value="CAP-07876" x="-25.4" y="95.504" size="1.778" layer="27" rot="R180" display="off"/>
 <attribute name="NAME" x="25.5778" y="48.8188" size="0.6096" layer="25" font="vector" rot="R180"/>
 </element>
-<element name="C7" library="SparkFun-Capacitors" package="0603-CAP" value="22pF" x="19.05" y="44.958" smashed="yes" rot="R90">
+<element name="C7" library="SparkFun-Capacitors" package="0603-CAP" value="18pF" x="19.05" y="44.958" smashed="yes" rot="R90">
 <attribute name="PROD_ID" value="CAP-07876" x="66.04" y="97.028" size="1.778" layer="27" rot="R90" display="off"/>
 <attribute name="NAME" x="17.9832" y="43.6118" size="0.6096" layer="25" font="vector" rot="R90"/>
@@
 <attribute name="NAME" x="45.4406" y="42.7482" size="0.6096" layer="25" font="vector"/>
 </element>
-<element name="C5" library="SparkFun-Passives" package="0603-CAP" value="4.7u" x="51.816" y="46.482" smashed="yes">
+<element name="C5" library="SparkFun-Passives" package="0603-CAP" value="4.7uF" x="51.816" y="46.482" smashed="yes">
 <attribute name="NAME" x="50.4698" y="47.2948" size="0.6096" layer="25" font="vector"/>
 </element>
-<element name="C8" library="SparkFun-Passives" package="0603-CAP" value="4.7u" x="38.1" y="43.18" smashed="yes" rot="R270">
+<element name="C8" library="SparkFun-Passives" package="0603-CAP" value="4.7uF" x="38.1" y="43.18" smashed="yes" rot="R270">
 <attribute name="NAME" x="37.846" y="46.2026" size="0.6096" layer="25" font="vector" rot="R270"/>
 </element>
